Commit message: Task A.3: Created a yaml file to provide a complete parametric description of a differential drive robot; modified the turtlebot3 URDF so that it uses the parameters.

File: nuturtle_description/urdf/turtlebot3_burger.urdf.xacro (robot description, xacro)
@@ -2,7 +2,15 @@
 <!-- Changed the name of the file to be turtlebot3_burger.urdf.xacro -->
 <!-- Changed every filename from turtlebot3_description to nuturtle_description and removed the subdirectories in /meshes -->
+<!-- Changed joint origins to use track_width parameter -->
+<!-- Changed joint origins to use wheel_radius parameter -->
+<!-- Changed the base_link's collision geometry from a box to a cylinder -->
 <robot name="turtlebot3_burger"
   xmlns:xacro="http://ros.org/wiki/xacro">
   <!-- <xacro:include filename="$(find nuturtle_description)/urdf/common_properties.urdf.xacro"/> -->
+  <xacro:property name="path_yaml" value="$(find nuturtle_description)/config/diff_params.yaml"/>
+  <xacro:property name="dict_yaml" value="${xacro.load_yaml(path_yaml)['/**']['ros__parameters']}"/>
+  <xacro:property name="wheel_radius" value="${dict_yaml['wheel_radius']}"/>
+  <xacro:property name="track_width" value="${dict_yaml['track_width']}"/>
+  <xacro:property name="collision_radius" value="${dict_yaml['collision_radius']}"/>
   <xacro:arg name="namespace" default=""/>
   <xacro:property name="namespace" value="$(arg namespace)"/>
@@ -55,5 +63,5 @@
       <origin xyz="-0.032 0 0.070" rpy="0 0 0"/>
       <geometry>
-        <box size="0.140 0.140 0.143"/>
+         <cylinder length="0.143" radius="${collision_radius}"/>
       </geometry>
     </collision>
@@ -67,5 +75,5 @@
     <parent link="${namespace}base_link"/>
     <child link="${namespace}wheel_left_link"/>
-    <origin xyz="0.0 0.08 0.023" rpy="-1.57 0 0"/>
+    <origin xyz="0.0 ${track_width/2} 0.023" rpy="-1.57 0 0"/>
     <axis xyz="0 0 1"/>
   </joint>
@@ -81,5 +89,5 @@
       <origin xyz="0 0 0" rpy="0 0 0"/>
       <geometry>
-        <cylinder length="0.018" radius="0.033"/>
+        <cylinder length="0.018" radius="${wheel_radius}"/>
       </geometry>
     </collision>
@@ -93,5 +101,5 @@
     <parent link="${namespace}base_link"/>
     <child link="${namespace}wheel_right_link"/>
-    <origin xyz="0.0 -0.080 0.023" rpy="-1.57 0 0"/>
+    <origin xyz="0.0 ${-track_width/2} 0.023" rpy="-1.57 0 0"/>
     <axis xyz="0 0 1"/>
   </joint>
@@ -107,5 +115,5 @@
       <origin xyz="0 0 0" rpy="0 0 0"/>
       <geometry>
-        <cylinder length="0.018" radius="0.033"/>
+        <cylinder length="0.018" radius="${wheel_radius}"/>
       </geometry>
     </collision>

Commit message: Task A.4: Modified load_one.launch.xml to take an argument called color and set the frame_prefix parameter of the robot_state_publisher.

File: nuturtle_description/urdf/turtlebot3_burger.urdf.xacro (robot description, xacro)
@@ -5,4 +5,6 @@
 <!-- Changed joint origins to use wheel_radius parameter -->
 <!-- Changed the base_link's collision geometry from a box to a cylinder -->
+<!-- Set the argument for colors -->
+<!-- Removed namespace argument and references -->
 <robot name="turtlebot3_burger"
   xmlns:xacro="http://ros.org/wiki/xacro">
@@ -13,15 +15,7 @@
   <xacro:property name="track_width" value="${dict_yaml['track_width']}"/>
   <xacro:property name="collision_radius" value="${dict_yaml['collision_radius']}"/>
-  <xacro:arg name="namespace" default=""/>
-  <xacro:property name="namespace" value="$(arg namespace)"/>
-  <!-- Init colour -->
-  <material name="black">
-      <color rgba="0.0 0.0 0.0 1.0"/>
-  </material>
-  <material name="dark">
-    <color rgba="0.3 0.3 0.3 1.0"/>
-  </material>
-  <material name="light_black">
-    <color rgba="0.4 0.4 0.4 1.0"/>
+  <xacro:arg name="color" default="purple"/>
+  <material name="purple">
+      <color rgba="0.3 0.16 0.52 1.0"/>
   </material>
   <material name="blue">
@@ -31,26 +25,14 @@
     <color rgba="0.0 0.8 0.0 1.0"/>
   </material>
-  <material name="grey">
-    <color rgba="0.5 0.5 0.5 1.0"/>
-  </material>
-  <material name="orange">
-    <color rgba="1.0 0.4235 0.0392 1.0"/>
-  </material>
-  <material name="brown">
-    <color rgba="0.8706 0.8118 0.7647 1.0"/>
-  </material>
   <material name="red">
     <color rgba="0.8 0.0 0.0 1.0"/>
   </material>
-  <material name="white">
-    <color rgba="1.0 1.0 1.0 1.0"/>
-  </material>
-  <link name="${namespace}base_footprint"/>
-  <joint name="${namespace}base_joint" type="fixed">
-    <parent link="${namespace}base_footprint"/>
-    <child link="${namespace}base_link"/>
+  <link name="base_footprint"/>
+  <joint name="base_joint" type="fixed">
+    <parent link="base_footprint"/>
+    <child link="base_link"/>
     <origin xyz="0.0 0.0 0.010" rpy="0 0 0"/>
   </joint>
-  <link name="${namespace}base_link">
+  <link name="base_link">
     <visual>
       <origin xyz="-0.032 0 0.0" rpy="0 0 0"/>
@@ -58,5 +40,5 @@
         <mesh filename="package://nuturtle_description/meshes/burger_base.stl" scale="0.001 0.001 0.001"/>
       </geometry>
-      <material name="light_black"/>
+      <material name="$(arg color)"/>
     </visual>
     <collision>
@@ -72,11 +54,11 @@
     </inertial>
   </link>
-  <joint name="${namespace}wheel_left_joint" type="continuous">
-    <parent link="${namespace}base_link"/>
-    <child link="${namespace}wheel_left_link"/>
+  <joint name="wheel_left_joint" type="continuous">
+    <parent link="base_link"/>
+    <child link="wheel_left_link"/>
     <origin xyz="0.0 ${track_width/2} 0.023" rpy="-1.57 0 0"/>
     <axis xyz="0 0 1"/>
   </joint>
-  <link name="${namespace}wheel_left_link">
+  <link name="wheel_left_link">
     <visual>
       <origin xyz="0 0 0" rpy="1.57 0 0"/>
@@ -84,5 +66,5 @@
         <mesh filename="package://nuturtle_description/meshes/left_tire.stl" scale="0.001 0.001 0.001"/>
       </geometry>
-      <material name="dark"/>
+      <material name="$(arg color)"/>
     </visual>
     <collision>
@@ -98,11 +80,11 @@
     </inertial>
   </link>
-  <joint name="${namespace}wheel_right_joint" type="continuous">
-    <parent link="${namespace}base_link"/>
-    <child link="${namespace}wheel_right_link"/>
+  <joint name="wheel_right_joint" type="continuous">
+    <parent link="base_link"/>
+    <child link="wheel_right_link"/>
     <origin xyz="0.0 ${-track_width/2} 0.023" rpy="-1.57 0 0"/>
     <axis xyz="0 0 1"/>
   </joint>
-  <link name="${namespace}wheel_right_link">
+  <link name="wheel_right_link">
     <visual>
       <origin xyz="0 0 0" rpy="1.57 0 0"/>
@@ -110,5 +92,5 @@
         <mesh filename="package://nuturtle_description/meshes/right_tire.stl" scale="0.001 0.001 0.001"/>
       </geometry>
-      <material name="dark"/>
+      <material name="$(arg color)"/>
     </visual>
     <collision>
@@ -124,10 +106,10 @@
     </inertial>
   </link>
-  <joint name="${namespace}caster_back_joint" type="fixed">
-    <parent link="${namespace}base_link"/>
-    <child link="${namespace}caster_back_link"/>
+  <joint name="caster_back_joint" type="fixed">
+    <parent link="base_link"/>
+    <child link="caster_back_link"/>
     <origin xyz="-0.081 0 -0.004" rpy="-1.57 0 0"/>
   </joint>
-  <link name="${namespace}caster_back_link">
+  <link name="caster_back_link">
     <collision>
       <origin xyz="0 0.001 0" rpy="0 0 0"/>
@@ -142,16 +124,16 @@
     </inertial>
   </link>
-  <joint name="${namespace}imu_joint" type="fixed">
-    <parent link="${namespace}base_link"/>
-    <child link="${namespace}imu_link"/>
+  <joint name="imu_joint" type="fixed">
+    <parent link="base_link"/>
+    <child link="imu_link"/>
     <origin xyz="-0.032 0 0.068" rpy="0 0 0"/>
   </joint>
-  <link name="${namespace}imu_link"/>
-  <joint name="${namespace}scan_joint" type="fixed">
-    <parent link="${namespace}base_link"/>
-    <child link="${namespace}base_scan"/>
+  <link name="imu_link"/>
+  <joint name="scan_joint" type="fixed">
+    <parent link="base_link"/>
+    <child link="base_scan"/>
     <origin xyz="-0.032 0 0.172" rpy="0 0 0"/>
   </joint>
-  <link name="${namespace}base_scan">
+  <link name="base_scan">
     <visual>
       <origin xyz="0 0 0.0" rpy="0 0 0"/>
@@ -159,5 +141,5 @@
         <mesh filename="package://nuturtle_description/meshes/lds.stl" scale="0.001 0.001 0.001"/>
       </geometry>
-      <material name="dark"/>
+      <material name="$(arg color)"/>
     </visual>
     <collision>
